File: PiPico_iCE40UL1K_Addon/PiPico_iCE40UL1K_Addon.kicad_sch (KiCad schematic)
At the start: 29 parts, among them J1 Conn_01x20_Pin, J2 Conn_01x20_Pin, SW1 SW_Push, U1 ICE40LP384-SG32, U2 TLV70033_SOT23-5, U3 TLV70025_SOT23-5, U4 TLV70012_SOT23-5

Commit message: Started XIAO breakout, did some basic floorplanning
Connections:
- net GND: now also U1.33
Changed lines of the file:
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@@
+	)
+	(label "GND"
+		(at 158.75 24.13 0)
+		(effects
+			(font
+				(size 1.27 1.27)
+			)
+			(justify left bottom)
+		)
 	)
 	(label "GND"
