File: Xiao_iCE40LP384_Addon/Xiao_iCE40LP384_Addon.kicad_pcb (KiCad board)
At the start: 4 copper layers, 17.8 x 21 mm, 42 parts, among them J1 Conn_01x07_Pin, J2 Conn_01x07_Pin, SW1 SW_Push, U1 ICE40LP384-SG32, U2 ADP322ACPZ-145-R7

Commit message: Slight improvements to ground
Routing:
- net /CDONE: track 32.1 -> 31.4 mm
- net /GND: vias 47 -> 48
Changed lines of the file:
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@@
+	)
+	(via
+		(at 114.7572 67.31)
+		(size 0.6)
+		(drill 0.3)
+		(layers "F.Cu" "B.Cu")
+		(free yes)
+		(net 2)
 	)
 	(via
@@
 	)
 	(segment
+		(start 108.443022 63.746001)
+		(end 107.9373 63.746001)
+		(width 0.2)
+		(layer "F.Cu")
+		(net 46)
+	)
+	(segment
+		(start 108.7666 64.1642)
+		(end 108.7628 64.1604)
+		(width 0.2)
+		(layer "F.Cu")
+		(net 46)
+	)
+	(segment
+		(start 109.8804 65.459074)
+		(end 109.8804 65.348078)
+		(width 0.2)
+		(layer "F.Cu")
+		(net 46)
+	)
+	(segment
+		(start 110.359726 65.9384)
+		(end 109.8804 65.459074)
+		(width 0.2)
+		(layer "F.Cu")
+		(net 46)
+	)
+	(segment
 		(start 101.346 53.6448)
 		(end 100.7364 53.0352)
@@
 	)
 	(segment
-		(start 113.3 67.15)
-		(end 112.0884 65.9384)
-		(width 0.2)
-		(layer "F.Cu")
-		(net 46)
-	)
-	(segment
-		(start 108.443022 63.746001)
-		(end 107.9373 63.746001)
-		(width 0.2)
-		(layer "F.Cu")
-		(net 46)
-	)
-	(segment
 		(start 101.346 53.7952)
 		(end 101.346 53.6448)
@@
 	)
 	(segment
-		(start 108.7666 64.1642)
-		(end 108.7628 64.1604)
+		(start 109.8804 65.348078)
+		(end 108.7666 64.234278)
+		(width 0.2)
+		(layer "F.Cu")
+		(net 46)
+	)
+	(segment
+		(start 112.0884 65.9384)
+		(end 110.359726 65.9384)
+		(width 0.2)
+		(layer "F.Cu")
+		(net 46)
+	)
+	(segment
+		(start 112.7506 66.6006)
+		(end 112.0884 65.9384)
+		(width 0.2)
+		(layer "F.Cu")
+		(net 46)
+	)
+	(segment
+		(start 112.7506 67.1068)
+		(end 112.7506 66.6006)
+		(width 0.2)
+		(layer "F.Cu")
+		(net 46)
+	)
+	(segment
+		(start 108.7628 64.065779)
+		(end 108.443022 63.746001)
+		(width 0.2)
+		(layer "F.Cu")
+		(net 46)
+	)
+	(segment
+		(start 108.7628 64.1604)
+		(end 108.7628 64.065779)
 		(width 0.2)
 		(layer "F.Cu")
@@
 		(net 46)
 	)
-	(segment
-		(start 108.7628 64.065779)
-		(end 108.443022 63.746001)
-		(width 0.2)
-		(layer "F.Cu")
+	(via
+		(at 112.7506 67.1068)
+		(size 0.6)
+		(drill 0.3)
+		(layers "F.Cu" "B.Cu")
 		(net 46)
 	)
-	(segment
-		(start 109.8804 65.348078)
-		(end 108.7666 64.234278)
-		(width 0.2)
-		(layer "F.Cu")
+	(via
+		(at 100.7364 53.0352)
+		(size 0.6)
+		(drill 0.3)
+		(layers "F.Cu" "B.Cu")
 		(net 46)
 	)
 	(segment
-		(start 108.7628 64.1604)
-		(end 108.7628 64.065779)
-		(width 0.2)
-		(layer "F.Cu")
+		(start 109.8296 66.294)
+		(end 108.0516 64.516)
+		(width 0.2)
+		(layer "B.Cu")
 		(net 46)
 	)
 	(segment
-		(start 109.8804 65.459074)
-		(end 109.8804 65.348078)
-		(width 0.2)
-		(layer "F.Cu")
-		(net 46)
-	)
-	(segment
-		(start 112.0884 65.9384)
-		(end 110.359726 65.9384)
-		(width 0.2)
-		(layer "F.Cu")
-		(net 46)
-	)
-	(segment
-		(start 110.359726 65.9384)
-		(end 109.8804 65.459074)
-		(width 0.2)
-		(layer "F.Cu")
-		(net 46)
-	)
-	(via
-		(at 113.3 67.15)
-		(size 0.6)
-		(drill 0.3)
-		(layers "F.Cu" "B.Cu")
-		(net 46)
-	)
-	(via
-		(at 100.7364 53.0352)
-		(size 0.6)
-		(drill 0.3)
-		(layers "F.Cu" "B.Cu")
+		(start 102.4128 64.0588)
+		(end 102.4128 58.166)
+		(width 0.2)
+		(layer "B.Cu")
 		(net 46)
 	)
@@
 	)
 	(segment
+		(start 100.7364 56.4896)
+		(end 100.7364 53.0352)
+		(width 0.2)
+		(layer "B.Cu")
+		(net 46)
+	)
+	(segment
+		(start 112.4966 67.5132)
+		(end 111.4552 67.5132)
+		(width 0.2)
+		(layer "B.Cu")
+		(net 46)
+	)
+	(segment
+		(start 112.7506 67.2592)
+		(end 112.4966 67.5132)
+		(width 0.2)
+		(layer "B.Cu")
+		(net 46)
+	)
+	(segment
+		(start 110.236 66.294)
+		(end 109.8296 66.294)
+		(width 0.2)
+		(layer "B.Cu")
+		(net 46)
+	)
+	(segment
+		(start 112.7506 67.1068)
+		(end 112.7506 67.2592)
+		(width 0.2)
+		(layer "B.Cu")
+		(net 46)
+	)
+	(segment
+		(start 102.4128 58.166)
+		(end 100.7364 56.4896)
+		(width 0.2)
+		(layer "B.Cu")
+		(net 46)
+	)
+	(segment
+		(start 111.4552 67.5132)
+		(end 110.236 66.294)
+		(width 0.2)
+		(layer "B.Cu")
+		(net 46)
+	)
+	(segment
 		(start 102.87 64.516)
 		(end 102.4128 64.0588)
 		(width 0.2)
 		(layer "B.Cu")
-		(net 46)
-	)
-	(segment
-		(start 110.236 66.294)
-		(end 109.8296 66.294)
-		(width 0.2)
-		(layer "B.Cu")
-		(net 46)
-	)
-	(segment
-		(start 112.9368 67.5132)
-		(end 111.4552 67.5132)
-		(width 0.2)
-		(layer "B.Cu")
-		(net 46)
-	)
-	(segment
-		(start 100.7364 56.4896)
-		(end 100.7364 53.0352)
-		(width 0.2)
-		(layer "B.Cu")
-		(net 46)
-	)
-	(segment
-		(start 102.4128 58.166)
-		(end 100.7364 56.4896)
-		(width 0.2)
-		(layer "B.Cu")
-		(net 46)
-	)
-	(segment
-		(start 109.8296 66.294)
-		(end 108.0516 64.516)
-		(width 0.2)
-		(layer "B.Cu")
-		(net 46)
-	)
-	(segment
-		(start 111.4552 67.5132)
-		(end 110.236 66.294)
-		(width 0.2)
-		(layer "B.Cu")
-		(net 46)
-	)
-	(segment
-		(start 113.3 67.15)
-		(end 112.9368 67.5132)
-		(width 0.2)
-		(layer "B.Cu")
-		(net 46)
-	)
-	(segment
-		(start 102.4128 64.0588)
-		(end 102.4128 58.166)
-		(width 0.2)
-		(layer "B.Cu")
